File: kicad/nano_dbg.sch (KiCad schematic (older format))
At the start: 22 parts, among them J3 USB_Micro, U12 MIC2877, U9 CP2102N-QFN20

Commit message: pmic_int connection
Parts:
- U9: footprint Package_DFN_QFN:SiliconLabs_QFN-20-1EP_3x3mm_P0.5mm_ThermalVias -> Custom Components:SiliconLabs_QFN-20-1EP_3x3mm_CUSTOM
Changed lines of the file:
@@
 F 0 "U9" H 5500 3815 50  0000 C CNN
 F 1 "CP2102N-QFN20" H 5500 3724 50  0000 C CNN
-F 2 "Package_DFN_QFN:SiliconLabs_QFN-20-1EP_3x3mm_P0.5mm_ThermalVias" H 5500 2950 50  0001 C CNN
+F 2 "Custom Components:SiliconLabs_QFN-20-1EP_3x3mm_CUSTOM" H 5500 2950 50  0001 C CNN
 F 3 "" H 5500 2950 50  0001 C CNN
 	1    5500 2750
